File: AnalogEVSE.kicad_pcb (KiCad board)
At the start: 2 copper layers, 102.3 x 84.5 mm, 78 parts, among them K1 Relay, P1 Pilot, P2 Rext, P3 230V, P4 Relay 1, P5 Status LEDs, P6 Power, P7 Relay 2, Q1 BC337-40, Q2 BC337-40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

Commit message: Update
Changed lines of the file:
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@@
   (segment (start 128.651 39.116) (end 128.27 38.735) (width 0.45) (layer B.Cu) (net 47))
   (segment (start 128.651 39.116) (end 128.27 38.735) (width 0.45) (layer B.Cu) (net 47))
-  (segment (start 92.329 41.783) (end 94.869 41.783) (width 0.45) (layer B.Cu) (net 48))
+  (segment (start 94.869 41.783) (end 92.329 41.783) (width 0.45) (layer B.Cu) (net 48))
   (segment (start 124.968 45.72) (end 126.111 45.72) (width 0.45) (layer B.Cu) (net 49))
   (segment (start 126.619 45.212) (end 128.524 45.212) (width 0.45) (layer B.Cu) (net 49))
