File: AnalogEVSE.sch (KiCad schematic (older format))
At the start: 70 parts, among them K1 Relay, P1 Pilot, P2 Rext, P3 230V, P4 Relay 1, P5 Status LEDs, P6 Power, P7 Relay 2, Q1 BC337-40, Q2 BC337-40, Q3 BC557, Q4 BC337-40, T1 12V/3VA, U1 LM2901, U2 LM7812, U3 LM7912, U4 LM2901

Commit message: Update
Parts:
- C1, C2, C5, C6, C7, C8, C9: symbol C -> C-RESCUE-AnalogEVSE
- C3, C4: symbol CP1 -> CP1-RESCUE-AnalogEVSE
- D10, D11, D12, D8: symbol LED -> LED-RESCUE-AnalogEVSE
- R1, R10, R11, R12, R13, R14, R15, R16, R17, R18, R19, R2, R20, R21, R22, R23, R24, R25, R26, R27, R28, R29, R3, R30, R4, R5, R6, R7, R8, R9: symbol R -> R-RESCUE-AnalogEVSE
- U1, U4: symbol LM339 -> LM339-RESCUE-AnalogEVSE
Changed lines of the file:
@@
 EESchema Schematic File Version 2
+LIBS:AnalogEVSE-rescue
 LIBS:power
 LIBS:device
@@
 LIBS:memory
 LIBS:xilinx
-LIBS:special
 LIBS:microcontrollers
 LIBS:dsp
@@
 $EndDescr
 $Comp
-L LM339 U1
+L LM339-RESCUE-AnalogEVSE U1
 U 2 1 56484E4A
 P 2850 3650
@@
 $EndComp
 $Comp
-L LM339 U1
+L LM339-RESCUE-AnalogEVSE U1
 U 1 1 56484E6B
 P 2850 4650
@@
 $EndComp
 $Comp
-L LM339 U1
+L LM339-RESCUE-AnalogEVSE U1
 U 4 1 56484E7B
 P 2850 5650
@@
 $EndComp
 $Comp
-L LM339 U1
+L LM339-RESCUE-AnalogEVSE U1
 U 3 1 56484E8A
 P 2850 6650
@@
 $EndComp
 $Comp
-L GND #PWR01
+L GND-RESCUE-AnalogEVSE #PWR01
 U 1 1 56484EF1
 P 1650 3150
@@
 $EndComp
 $Comp
-L R R5
+L R-RESCUE-AnalogEVSE R5
 U 1 1 5648522E
 P 2850 3050
@@
 $EndComp
 $Comp
-L C C1
+L C-RESCUE-AnalogEVSE C1
 U 1 1 56485246
 P 1300 3950
@@
 $EndComp
 $Comp
-L R R4
+L R-RESCUE-AnalogEVSE R4
 U 1 1 56485307
 P 2000 3050
@@
 $EndComp
 $Comp
-L R R7
+L R-RESCUE-AnalogEVSE R7
 U 1 1 56485346
 P 3650 3400
@@
 $EndComp
 $Comp
-L GND #PWR011
+L GND-RESCUE-AnalogEVSE #PWR011
 U 1 1 564853A0
 P 1300 4150
@@
 $EndComp
 $Comp
-L R R6
+L R-RESCUE-AnalogEVSE R6
 U 1 1 564853D7
 P 3350 4400
@@
 $EndComp
 $Comp
-L R R8
+L R-RESCUE-AnalogEVSE R8
 U 1 1 56485419
 P 3950 4400
@@
 $EndComp
 $Comp
-L R R9
+L R-RESCUE-AnalogEVSE R9
 U 1 1 56485490
 P 4500 5100
@@
 $EndComp
 $Comp
-L R R10
+L R-RESCUE-AnalogEVSE R10
 U 1 1 564854A1
 P 4750 4850
@@
 $EndComp
 $Comp
-L R R1
+L R-RESCUE-AnalogEVSE R1
 U 1 1 564854AC
 P 1850 4500
@@
 $EndComp
 $Comp
-L R R2
+L R-RESCUE-AnalogEVSE R2
 U 1 1 564854B2
 P 1850 5000
@@
 $EndComp
 $Comp
-L R R3
+L R-RESCUE-AnalogEVSE R3
 U 1 1 564854B8
 P 1850 5500
@@
 $EndComp
 $Comp
-L C C2
+L C-RESCUE-AnalogEVSE C2
 U 1 1 564854BE
 P 2100 4950
@@
 $EndComp
 $Comp
-L GND #PWR016
+L GND-RESCUE-AnalogEVSE #PWR016
 U 1 1 564854C4
 P 2100 5150
@@
 $EndComp
 $Comp
-L GND #PWR019
+L GND-RESCUE-AnalogEVSE #PWR019
 U 1 1 56485718
 P 2900 1300
@@
 $EndComp
 $Comp
-L CP1 C3
+L CP1-RESCUE-AnalogEVSE C3
 U 1 1 56485720
 P 3600 1000
@@
 $EndComp
 $Comp
-L CP1 C4
+L CP1-RESCUE-AnalogEVSE C4
 U 1 1 5648572D
 P 3600 1400
@@
 $EndComp
 $Comp
-L C C6
+L C-RESCUE-AnalogEVSE C6
 U 1 1 5648597D
 P 5100 1000
@@
 $EndComp
 $Comp
-L C C7
+L C-RESCUE-AnalogEVSE C7
 U 1 1 56485983
 P 5100 1500
@@
 $EndComp
 $Comp
-L R R14
+L R-RESCUE-AnalogEVSE R14
 U 1 1 56485D3D
 P 5650 800
@@
 $EndComp
 $Comp
-L R R15
+L R-RESCUE-AnalogEVSE R15
 U 1 1 56485D43
 P 6150 800
@@
 $EndComp
 $Comp
-L R R16
+L R-RESCUE-AnalogEVSE R16
 U 1 1 56485D49
 P 6650 800
@@
 $EndComp
 $Comp
-L R R17
+L R-RESCUE-AnalogEVSE R17
 U 1 1 56485D4F
 P 7150 800
@@
 $EndComp
 $Comp
-L R R18
+L R-RESCUE-AnalogEVSE R18
 U 1 1 56485D55
 P 7650 800
@@
 Vneg
 $Comp
-L C C5
+L C-RESCUE-AnalogEVSE C5
 U 1 1 56485F71
 P 5000 7200
@@
 $EndComp
 $Comp
-L R R12
+L R-RESCUE-AnalogEVSE R12
 U 1 1 56485F77
 P 4750 7250
@@
 $EndComp
 $Comp
-L GND #PWR022
+L GND-RESCUE-AnalogEVSE #PWR022
 U 1 1 56485F87
 P 4750 7600
@@
 $EndComp
 $Comp
-L R R11
+L R-RESCUE-AnalogEVSE R11
 U 1 1 564861D6
 P 4750 6400
@@
 $EndComp
 $Comp
-L GND #PWR023
+L GND-RESCUE-AnalogEVSE #PWR023
 U 1 1 564861DC
 P 4750 6650
@@
 $EndComp
 $Comp
-L C C8
+L C-RESCUE-AnalogEVSE C8
 U 1 1 56486234
 P 5750 5050
@@
 $EndComp
 $Comp
-L R R13
+L R-RESCUE-AnalogEVSE R13
 U 1 1 5648623A
 P 5500 5100
@@
 $EndComp
 $Comp
-L GND #PWR024
+L GND-RESCUE-AnalogEVSE #PWR024
 U 1 1 56486240
 P 5500 5450
@@
 $EndComp
 $Comp
-L LM339 U4
+L LM339-RESCUE-AnalogEVSE U4
 U 2 1 564863A9
 P 7050 3050
@@
 $EndComp
 $Comp
-L LM339 U4
+L LM339-RESCUE-AnalogEVSE U4
 U 1 1 564863B8
 P 7050 3900
@@
 $EndComp
 $Comp
-L LM339 U4
+L LM339-RESCUE-AnalogEVSE U4
 U 4 1 564863C7
 P 7050 4750
@@
 $EndComp
 $Comp
-L LM339 U4
+L LM339-RESCUE-AnalogEVSE U4
 U 3 1 564863D6
 P 7050 5600
@@
 $EndComp
 $Comp
-L GND #PWR033
+L GND-RESCUE-AnalogEVSE #PWR033
 U 1 1 5648678C
 P 1500 2350
@@
 $EndComp
 $Comp
-L R R25
+L R-RESCUE-AnalogEVSE R25
 U 1 1 56486B7F
 P 9650 6300
@@
 $EndComp
 $Comp
-L R R21
+L R-RESCUE-AnalogEVSE R21
 U 1 1 5648DDB8
 P 9350 4950
@@
 $EndComp
 $Comp
-L R R24
+L R-RESCUE-AnalogEVSE R24
 U 1 1 5648DDC3
 P 9800 5600
@@
 $EndComp
 $Comp
-L R R23
+L R-RESCUE-AnalogEVSE R23
 U 1 1 5648DFD3
 P 9800 4450
@@
 $EndComp
 $Comp
-L R R20
+L R-RESCUE-AnalogEVSE R20
 U 1 1 5648E221
 P 8950 4500
@@
 $EndComp
 $Comp
-L R R19
+L R-RESCUE-AnalogEVSE R19
 U 1 1 5648E2D7
 P 8050 2800
@@
 $EndComp
 $Comp
-L C C9
+L C-RESCUE-AnalogEVSE C9
 U 1 1 5648E2DD
 P 8050 3250
@@
 $EndComp
 $Comp
-L GND #PWR038
+L GND-RESCUE-AnalogEVSE #PWR038
 U 1 1 5648E2FC
 P 8050 3450
@@
 $EndComp
 $Comp
-L GND #PWR040
+L GND-RESCUE-AnalogEVSE #PWR040
 U 1 1 5648E322
 P 9050 3650
@@
 $EndComp
 $Comp
-L R R22
+L R-RESCUE-AnalogEVSE R22
 U 1 1 5648E445
 P 9800 2850
@@
 $EndComp
 $Comp
-L R R26
+L R-RESCUE-AnalogEVSE R26
 U 1 1 565E00E5
 P 9550 3450
@@
 -Waiting
 $Comp
-L R R27
+L R-RESCUE-AnalogEVSE R27
 U 1 1 56C4CAED
 P 1300 3400
@@
 Error
 $Comp
-L LED D10
+L LED-RESCUE-AnalogEVSE D10
 U 1 1 5738428E
 P 10150 6050
@@
 	9900 6300 10550 6300
 $Comp
-L R R28
+L R-RESCUE-AnalogEVSE R28
 U 1 1 5738EB39
 P 9650 6050
@@
 Connection ~ 9350 6300
 $Comp
-L GND #PWR042
+L GND-RESCUE-AnalogEVSE #PWR042
 U 1 1 57390357
 P 10400 6150
@@
 	9300 2000 9400 2000
 $Comp
-L LED D8
+L LED-RESCUE-AnalogEVSE D8
 U 1 1 5742CB96
 P 9050 3450
@@
 $EndComp
 $Comp
-L R R30
+L R-RESCUE-AnalogEVSE R30
 U 1 1 5741FA7A
 P 8600 5600
@@
 $EndComp
 $Comp
-L LED D12
+L LED-RESCUE-AnalogEVSE D12
 U 1 1 5741FB99
 P 8150 5600
@@
 Connection ~ 8950 5600
 $Comp
-L R R29
+L R-RESCUE-AnalogEVSE R29
 U 1 1 57421CE5
 P 8600 4100
@@
 $EndComp
 $Comp
-L LED D11
+L LED-RESCUE-AnalogEVSE D11
 U 1 1 57421CEB
 P 8150 4100
