File: AnalogEVSE.sch (KiCad schematic (older format))
At the start: 70 parts, among them K1 Relay, P1 Pilot, P2 Rext, P3 230V, P4 Relay 1, P5 Status LEDs, P6 Power, P7 Relay 2, Q1 BC337-40, Q2 BC337-40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

Commit message: Filter caps
Parts:
- removed C9: 1u/16V, mylib:C2, symbol C-RESCUE-AnalogEVSE
- added C10: 47n, mylib:C2, symbol C-RESCUE-AnalogEVSE
- added C9: 4u7/16V, mylib:C4, symbol CP1-RESCUE-AnalogEVSE
- U2: footprint mylib:7812 -> mylib:LM7812
- U3: footprint mylib:7912 -> mylib:LM7912
Connections:
- net +12V: now also C10.2
- net -12V: now also C10.1, C9.2
- net at D6.1 (A), Q2.2 (B), R19.1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: now also C9.1

Commit message: Stash
Parts:
- removed P7: Relay 2, mylib:Term-2pin, symbol CONN_2
- added P7: Relay 2, mylib:Term-3pin, symbol CONN_3
Connections:
- net at K1.12 (C2): now also P7.1 (P1)
- net at K1.14 (R2): now also P7.2 (PM)
- net at K1.16 (T2): now also P7.3 (P3)
Changed lines of the file:
@@
-$EndComp
-$Comp
-L CONN_2 P7
-U 1 1 56486B79
-P 10900 1300
-F 0 "P7" V 10850 1300 40  0000 C CNN
-F 1 "Relay 2" V 10950 1300 40  0000 C CNN
-F 2 "mylib:Term-2pin" H 10900 1300 60  0001 C CNN
-F 3 "" H 10900 1300 60  0000 C CNN
-	1    10900 1300
-	1    0    0    -1
 $EndComp
 $Comp
@@
 U 1 1 57272B9C
 P 10900 2950
-F 0 "P5" H 10850 2950 50  0000 L CNN
+F 0 "P5" H 10850 2950 40  0000 L CNN
 F 1 "Status LEDs" H 10750 2700 40  0000 L CNN
 F 2 "mylib:Term-3pin" H 10900 2950 60  0001 C CNN
@@
 	5350 1400 5350 1700
 Connection ~ 5350 1700
+$Comp
+L CONN_3 P7
+U 1 1 5755526C
+P 10900 1300
+F 0 "P7" V 10850 1250 40  0000 L CNN
+F 1 "Relay 2" V 10950 1200 40  0000 L CNN
+F 2 "mylib:Term-3pin" H 10900 1300 60  0001 C CNN
+F 3 "" H 10900 1300 60  0000 C CNN
+	1    10900 1300
+	1    0    0    -1
+$EndComp
+Wire Wire Line
+	10550 1300 10250 1300
+Wire Wire Line
+	10250 1300 10250 1400
+Wire Wire Line
+	10250 1400 10200 1400
 $EndSCHEMATC

Commit message: RV2
Parts:
- added RV2: 10k, mylib:Trimpot, symbol POT
Connections:
- net at C2.1, P2.1 (P1), R1.1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: now also RV2.1, RV2.2
- net at P2.2 (PM), R2.1, R3.2: now also RV2.3

Commit message: RV2
Parts:
- RV2: footprint mylib:Trimpot -> mylib:Trimpot2

Commit message: RV2
Parts:
- C10: value 47n -> 150n
Changed lines of the file:
@@
 P 5350 1200
 F 0 "C10" H 5350 1300 40  0000 L CNN
-F 1 "47n" H 5356 1115 40  0000 L CNN
+F 1 "150n" H 5356 1115 40  0000 L CNN
 F 2 "mylib:C2" H 5388 1050 30  0001 C CNN
 F 3 "~" H 5350 1200 60  0000 C CNN

Commit message: Aetzwerk
Parts:
- C3, C4: footprint mylib:C3 -> mylib:C5
- C9: footprint mylib:C4 -> mylib:C6
- RV2: footprint mylib:Trimpot2 -> mylib:Trimpot3
Changed lines of the file:
@@
 Sheet 1 1
 Title "AnalogEVSE"
-Date "2016-04-24"
-Rev "1.7"
+Date "2016-07-06"
+Rev "1.8"
 Comp ""
 Comment1 "Analog J1772 charge controller"
@@
 F 0 "C3" H 3650 1100 50  0000 L CNN
 F 1 "220u/25V" H 3200 900 50  0000 L CNN
-F 2 "mylib:C3" H 3600 1000 60  0001 C CNN
+F 2 "mylib:C5" H 3600 1000 60  0001 C CNN
 F 3 "~" H 3600 1000 60  0000 C CNN
 	1    3600 1000
@@
 F 0 "C4" H 3650 1500 50  0000 L CNN
 F 1 "220u/25V" H 3650 1300 50  0000 L CNN
-F 2 "mylib:C3" H 3600 1400 60  0001 C CNN
+F 2 "mylib:C5" H 3600 1400 60  0001 C CNN
 F 3 "~" H 3600 1400 60  0000 C CNN
 	1    3600 1400
@@
 F 0 "C9" H 8100 3350 50  0000 L CNN
 F 1 "4u7/16V" H 8100 3150 50  0000 L CNN
-F 2 "mylib:C4" H 8050 3250 60  0001 C CNN
+F 2 "mylib:C6" H 8050 3250 60  0001 C CNN
 F 3 "~" H 8050 3250 60  0000 C CNN
 	1    8050 3250
@@
 F 0 "RV2" H 1500 4900 50  0000 C CNN
 F 1 "10k" H 1500 5000 50  0000 C CNN
-F 2 "mylib:Trimpot2" H 1500 5000 60  0001 C CNN
+F 2 "mylib:Trimpot3" H 1500 5000 60  0001 C CNN
 F 3 "~" H 1500 5000 60  0000 C CNN
 	1    1500 5000

Commit message: Addition of C11
Parts:
- added C11: 220u/16V, mylib:C6, symbol CP1-RESCUE-AnalogEVSE
- R14: value 3k3 -> 4k7
- R15: value 2k7 -> 3k3
- R16: value 2k2 -> 5k6
- RV1, RV2: symbol POT -> POT-RESCUE-AnalogEVSE
Connections:
- net +12V: now also C11.1
- net at D7.1 (A), K1.8, Q2.3 (C)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: now also C11.2
